File: solar_necklace_2/lightsaber_necklace.kicad_sch (KiCad schematic)
At the start: 39 parts, among them J1 earring_mount, J2 earring_mount, J3 pins, J4 pins, Q1 dual_NMOS, Q2 dual_NMOS, Q3 dual_NMOS, Q4 AO3401A, U1 MCP1643xMS, U2 ATtiny416-M

Commit message: upload schematics
Connections:
- net LEDPOWA: no longer U2.10 (PB4)
- no-connect marks 14 -> 16
Other:
- note added: "After top layer PCB assembly 1. Solder LEDs 2. Program and test MCU (with EN switch off) 3. Apply conformal coating (not through holes), to earring basket, solar panel edge 4. Solder solar panel 5. Solder earring in with silver solder. 6. Apply conformal coating to earring on backside It is must harder to program the MCU once earring and capacitors are in place, so make sure you like the program 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"
- note removed: "After top layer PCB assembly 1. Solder LEDs 2. Program and test MCU (with EN switch off) 3. Apply conformal coating (not through holes), to earring basket, solar panel edge 4. Solder solar panel 5. Solder earring in with silver solder 6. Apply conformal coating to earring on backside 7. Solder capacitors"
Changed lines of the file:
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@@
   )
   (no_connect (at 254 133.35))
+  (no_connect (at 254 151.13))
+  (no_connect (at 262.89 151.13))
   (no_connect (at 254 143.51))
   (no_connect (at 31.75 66.04))
@@
     (effects (font (size 1.27 1.27)) (justify left bottom))
   )
-  (text "After top layer PCB assembly\n1. Solder LEDs\n2. Program and test MCU (with EN switch off)\n3. Apply conformal coating (not through holes), to earring basket, solar panel edge\n4. Solder solar panel\n5. Solder earring in with silver solder\n6. Apply conformal coating to earring on backside\n7. Solder capacitors"
-    (at 162.56 97.79 0)
+  (text "After top layer PCB assembly\n1. Solder LEDs\n2. Program and test MCU (with EN switch off)\n3. Apply conformal coating (not through holes), to earring basket, solar panel edge\n4. Solder solar panel\n5. Solder earring in with silver solder.\n6. Apply conformal coating to earring on backside\nIt is must harder to program the MCU once earring and capacitors are in place, so make sure you like the program first\n7. Solder capacitors"
+    (at 151.13 101.6 0)
     (effects (font (size 1.27 1.27)) (justify left bottom))
   )
@@
     )
   )
-  (global_label "LEDPOWA" (shape input) (at 254 151.13 0) (fields_autoplaced)
+  (global_label "LEDPOWA" (shape input) (at 262.89 151.13 0) (fields_autoplaced)
     (effects (font (size 1.27 1.27)) (justify left))
-    (property "Intersheetrefs" "${INTERSHEET_REFS}" (at 265.5728 151.13 0)
+    (property "Intersheetrefs" "${INTERSHEET_REFS}" (at 274.4628 151.13 0)
       (effects (font (size 1.27 1.27)) (justify left) hide)
     )
